File: imix.brd (EAGLE design)
At the start: 87 x 102.5 mm, 160 parts, among them Q1 AO3418, Q2 AO3415, Q3 AO3415, Q4 AO3415, Q5 AO3415, U1 BQ2423X, U10 ISL29035, U11 FX0S8700CQ, U3 AD712R, U4 AD712R, U5 LDO-TPS78233, U6 ATSAM4LCX_100, U8 SI7021, U9 NRF51822, X1 16MHz, X2 16MHz, X3 16MHz

Commit message: Prototype ready for final review and manufacture
Parts:
- removed DT10: CGRM4001-G, diode:SOD-123_MINI-SMA
- removed DT6, DT7: 16V, SparkFun-DiscreteSemi:SOD-123
- removed DT9: (no value), SparkFun-DiscreteSemi:SOD-123
- removed LED7: 3.3V, SparkFun-LED:LED-0603
- added D5: MBR0530, SparkFun-DiscreteSemi:SOD-123
- added D6: MBR0530, imix_v1:SOD-123
- added F5, F6: FIDUCIAL, GeekAmmo:FIDUCIAL
- added LED5: USER, SparkFun-LED:LED-0603
- added R30: 10K, SparkFun-Resistors:0603-RES
- BAT1: device SparkFun-Electromechanical:BATTERY_18650-HOLDER -> imix_v1:BATTERY_18650-HOLDER
- C10, C45, C8, C9, R11, R12, R4, R5, R6, R7, R8: value (none) -> DNP
- C11: value (none) -> 22pF
- C44, C46, C47, C7: value (none) -> 0.47uF
- C48: value (none) -> 4.7uF
- LED3: value NRF -> 3.3V
- LED4: value USER -> NRF
- R10, R13, R9: value (none) -> 10K
- R14: value (none) -> 2.2M
- R15: value (none) -> 160K
- U12: value TPS61040 -> 296-12686-1-ND
- U3: value AD712R -> TLV3202
- U4: value AD712R -> LM358
- moved LED3 64.0 mm to (3.00, 41.5), turned to 90 degrees
- moved LED4 43.3 mm to (52.8, 1.38)
- moved R13 5.78 mm to (76.0, 73.6), turned to 90 degrees
- moved C47 5.15 mm to (80.5, 77.5), flipped to the top, turned to 0 degrees
- moved C49 1.00 mm to (80.1, 73.7)
- moved BAT1 0.50 mm to (9.50, 35.0), flipped to the top
- renumbered DT5 to D4, U$2 to F1, U$3 to F3, U$5 to F4, U$6 to F2, U$7 to U12
Connections:
- net GND: now also D5.C, LED5.C, R30.1; no longer DT9.C, LED7.C
- net N$29: now also LED5.A; no longer LED4.A
- net N$38: now also LED3.A; no longer LED7.A
- net N$43: now also D6.A; no longer DT10.A
- net N$51: no longer DT6.C
- net N$52: no longer DT7.C
- net N$66: now also D5.A; no longer DT9.A
- net N$75: now also LED4.A; no longer LED3.A
- net NOISE1: no longer DT6.A
- net NOISE2: no longer DT7.A
- net TRNG_EN: now also R30.2
- net VHIGH: now also D6.C; no longer DT10.C
Routing:
- net GND: track 154.4 -> 166.1 mm
- net NOISE2: track 41.3 -> 32.3 mm
- net VHIGH: track 64.1 -> 57.3 mm, vias 5 -> 4
- net N$66: track 42.8 -> 46.3 mm
- net N$52: track 19.3 -> 17.0 mm
- net NOISE1: track 39.3 -> 37.1 mm
- net TRNG_EN: track 60.8 -> 62.5 mm, vias 3 -> 4
- net N$68: track 12.7 -> 11.4 mm
- net VCC_SENSE_3V3: track 90.2 -> 91.4 mm
- net USART2_TX: track 33.0 -> 31.9 mm
Other:
- board text added: "B2"
- board text added: "BATT CLIP"
- board text added: "D1"
- board text added: "DBG USB"
- board text added: "DNP"
- board text added: "F1"
- board text added: "F2"
- board text added: "F3"
- board text added: "F4"
- board text added: "F5"
- board text added: "F6"
- board text added: "J1"
- board text added: "J2"
- board text added: "J3"
- board text added: "J4"
- board text added: "J5"
- board text added: "J6"
- board text added: "J7"
- board text added: "LED1"
- board text added: "LED2"
- board text added: "LED3"
- board text added: "LED4"
- board text added: "LED5"
- board text added: "PCB Bottom"
- board text added: "PCB Top"
- board text added: "PWR MEAS"
- board text added: "R30"
- board text added: "SW1"
- board text added: "SW2"
- board text added: "TARGET USB"
- board text added: "U10"
- board text added: "U11"
- board text added: "U12"
- board text added: "U2"
- board text added: "U6"
- board text added: "U7"
- board text added: "U8"
- board text added: "U9"
- board text removed: "AT86RF233"
- board text removed: "DEBUG"
- board text removed: "FT231X"
- board text removed: "FX0S8700CQ"
- board text removed: "IC2"
- board text removed: "ISL29035"
- board text removed: "NRF51822"
- board text removed: "POWER MEASURE"
- board text removed: "SI7021"
