File: imix.sch (EAGLE design)
At the start: 160 parts, among them Q1 AO3418, Q2 AO3415, Q3 AO3415, Q4 AO3415, Q5 AO3415, U1 BQ2423X, U10 ISL29035, U11 FX0S8700CQ, U3 AD712R, U4 AD712R, U5 LDO-TPS78233, U6 ATSAM4LCX_100, U8 SI7021, U9 NRF51822, X1 16MHz, X2 16MHz, X4 16MHz

Commit message: Update component naming for consistency
Parts:
- removed X4: 16MHz, stanford_iot_research:XTAL_GROUNDED5X3.2MM
- added X3: 16MHz, stanford_iot_research:XTAL_GROUNDED5X3.2MM
- C49: value (none) -> 10uF
- L3: value (none) -> 10uH
Connections:
- net GND: now also X3.CASE; no longer X4.CASE
- net N$11: now also X2.1; no longer X1.1
- net N$13: now also X2.2; no longer X1.2
- net N$4: now also X1.1; no longer X4.1
- net N$40: now also X1.2; no longer X4.2
- net N$7: now also X3.2; no longer X2.2
- net N$9: now also X3.1; no longer X2.1
Changed lines of the file:
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@@
 <part name="GND37" library="SparkFun-Aesthetics" deviceset="DGND" device=""/>
 <part name="R3" library="SparkFun-Passives" deviceset="RESISTOR" device="0603-RES" value="10K"/>
-<part name="X1" library="stanford_iot_research" deviceset="XTAL_GROUNDED" device="5X3.2MM" value="16MHz"/>
+<part name="X2" library="stanford_iot_research" deviceset="XTAL_GROUNDED" device="5X3.2MM" value="16MHz"/>
 <part name="D8" library="SparkFun-DiscreteSemi" deviceset="DIODE" device="SOD523" value="1N4148XTPMSCT-ND"/>
 <part name="R26" library="SparkFun-Passives" deviceset="RESISTOR" device="0603-RES" value="10K"/>
@@
 <part name="C12" library="rcl" deviceset="C-EU" device="C0603" value="13pF"/>
 <part name="C6" library="rcl" deviceset="C-EU" device="C0603" value="13pF"/>
-<part name="X4" library="stanford_iot_research" deviceset="XTAL_GROUNDED" device="5X3.2MM" value="16MHz"/>
+<part name="X1" library="stanford_iot_research" deviceset="XTAL_GROUNDED" device="5X3.2MM" value="16MHz"/>
 <part name="U2" library="stanford_iot_research" deviceset="AT86RF233" device=""/>
 <part name="C32" library="rcl" deviceset="C-EU" device="C0603" value="100 nF"/>
@@
 <part name="GND24" library="SparkFun-Aesthetics" deviceset="DGND" device=""/>
 <part name="GND42" library="SparkFun-Aesthetics" deviceset="DGND" device=""/>
-<part name="X2" library="stanford_iot_research" deviceset="XTAL_GROUNDED" device="5X3.2MM" value="16MHz"/>
+<part name="X3" library="stanford_iot_research" deviceset="XTAL_GROUNDED" device="5X3.2MM" value="16MHz"/>
 <part name="GND43" library="SparkFun-Aesthetics" deviceset="DGND" device=""/>
 <part name="GND4" library="SparkFun-Aesthetics" deviceset="DGND" device=""/>
@@
 <part name="R37" library="SparkFun-Passives" deviceset="RESISTOR" device="0603-RES" value="4.7K"/>
 <part name="U$7" library="SparkFun-PowerIC" deviceset="TPS61040" device=""/>
-<part name="L3" library="SparkFun-Passives" deviceset="INDUCTOR" device="0805"/>
+<part name="L3" library="SparkFun-Passives" deviceset="INDUCTOR" device="0805" value="10uH"/>
 <part name="DT10" library="diode" deviceset="CGRM400*-G" device="" technology="1"/>
 <part name="R14" library="SparkFun-Resistors" deviceset="0.27OHM-1/10W-1%(0603)" device=""/>
@@
 <part name="C48" library="SparkFun-Capacitors" deviceset="CAP" device="0603-CAP"/>
 <part name="GND40" library="SparkFun-Aesthetics" deviceset="GND" device=""/>
-<part name="C49" library="SparkFun-Capacitors" deviceset="CAP_POL" device="C"/>
+<part name="C49" library="SparkFun-Capacitors" deviceset="CAP_POL" device="C" value="10uF"/>
 <part name="SJ6" library="SparkFun-Retired" deviceset="SOLDERJUMPER" device="NO"/>
 <part name="R11" library="SparkFun-Resistors" deviceset="0.27OHM-1/10W-1%(0603)" device=""/>
@@
 <instance part="GND37" gate="G$1" x="269.24" y="68.58"/>
 <instance part="R3" gate="G$1" x="269.24" y="99.06" rot="R90"/>
-<instance part="X1" gate="G$1" x="152.4" y="134.62" smashed="yes" rot="R90">
+<instance part="X2" gate="G$1" x="152.4" y="134.62" smashed="yes" rot="R90">
 <attribute name="NAME" x="146.558" y="136.398" size="1.778" layer="95" font="vector" rot="R180"/>
 <attribute name="VALUE" x="161.798" y="136.398" size="1.778" layer="95" font="vector" rot="R180"/>
@@
 <junction x="162.56" y="129.54"/>
 <wire x1="162.56" y1="124.46" x2="162.56" y2="129.54" width="0.1524" layer="91"/>
-<pinref part="X1" gate="G$1" pin="CASE"/>
+<pinref part="X2" gate="G$1" pin="CASE"/>
 <wire x1="157.48" y1="137.16" x2="162.56" y2="137.16" width="0.1524" layer="91"/>
 <junction x="162.56" y="137.16"/>
@@
 <pinref part="C24" gate="G$1" pin="1"/>
 <wire x1="152.4" y1="129.54" x2="149.86" y2="129.54" width="0.1524" layer="91"/>
-<pinref part="X1" gate="G$1" pin="1"/>
+<pinref part="X2" gate="G$1" pin="1"/>
 <wire x1="119.38" y1="129.54" x2="149.86" y2="129.54" width="0.1524" layer="91"/>
 <junction x="149.86" y="129.54"/>
@@
 <segment>
 <pinref part="C23" gate="G$1" pin="1"/>
-<pinref part="X1" gate="G$1" pin="2"/>
+<pinref part="X2" gate="G$1" pin="2"/>
 <wire x1="149.86" y1="144.78" x2="152.4" y2="144.78" width="0.1524" layer="91"/>
 <wire x1="119.38" y1="132.08" x2="132.08" y2="132.08" width="0.1524" layer="91"/>
@@
 <attribute name="VALUE" x="66.548" y="73.787" size="1.778" layer="96" rot="R180"/>
 </instance>
-<instance part="X4" gate="G$1" x="66.04" y="63.5" smashed="yes" rot="R270">
+<instance part="X1" gate="G$1" x="66.04" y="63.5" smashed="yes" rot="R270">
 <attribute name="NAME" x="59.944" y="62.23" size="1.778" layer="95" font="vector"/>
 <attribute name="VALUE" x="57.658" y="58.42" size="1.778" layer="95" font="vector"/>
@@
 <wire x1="68.58" y1="50.8" x2="63.5" y2="50.8" width="0.1524" layer="91"/>
 <wire x1="68.58" y1="50.8" x2="68.58" y2="53.34" width="0.1524" layer="91"/>
-<pinref part="X4" gate="G$1" pin="2"/>
+<pinref part="X1" gate="G$1" pin="2"/>
 <pinref part="U2" gate="G$1" pin="XTAL2"/>
 <wire x1="68.58" y1="50.8" x2="81.28" y2="50.8" width="0.1524" layer="91"/>
@@
 <wire x1="68.58" y1="71.12" x2="63.5" y2="71.12" width="0.1524" layer="91"/>
 <wire x1="68.58" y1="68.58" x2="68.58" y2="71.12" width="0.1524" layer="91"/>
-<pinref part="X4" gate="G$1" pin="1"/>
+<pinref part="X1" gate="G$1" pin="1"/>
 <wire x1="76.2" y1="71.12" x2="68.58" y2="71.12" width="0.1524" layer="91"/>
 <junction x="68.58" y="71.12"/>
@@
 </segment>
 <segment>
-<pinref part="X4" gate="G$1" pin="CASE"/>
+<pinref part="X1" gate="G$1" pin="CASE"/>
 <wire x1="60.96" y1="60.96" x2="53.34" y2="60.96" width="0.1524" layer="91"/>
 <wire x1="53.34" y1="60.96" x2="53.34" y2="50.8" width="0.1524" layer="91"/>
@@
 <instance part="GND24" gate="G$1" x="71.12" y="251.46" rot="R270"/>
 <instance part="GND42" gate="G$1" x="71.12" y="200.66"/>
-<instance part="X2" gate="G$1" x="73.66" y="271.78" rot="R270"/>
+<instance part="X3" gate="G$1" x="73.66" y="271.78" rot="R270"/>
 <instance part="GND43" gate="G$1" x="55.88" y="269.24" rot="R270"/>
 <instance part="R34" gate="G$1" x="162.56" y="223.52" rot="MR270"/>
@@
 </segment>
 <segment>
-<pinref part="X2" gate="G$1" pin="CASE"/>
+<pinref part="X3" gate="G$1" pin="CASE"/>
 <pinref part="GND43" gate="G$1" pin="GND"/>
 <wire x1="68.58" y1="269.24" x2="58.42" y2="269.24" width="0.1524" layer="91"/>
@@
 <pinref part="C34" gate="G$1" pin="2"/>
 <wire x1="101.6" y1="259.08" x2="76.2" y2="259.08" width="0.1524" layer="91"/>
-<pinref part="X2" gate="G$1" pin="2"/>
+<pinref part="X3" gate="G$1" pin="2"/>
 <wire x1="76.2" y1="259.08" x2="71.12" y2="259.08" width="0.1524" layer="91"/>
 <wire x1="76.2" y1="261.62" x2="76.2" y2="259.08" width="0.1524" layer="91"/>
@@
 <pinref part="C39" gate="G$1" pin="2"/>
 <wire x1="83.82" y1="279.4" x2="76.2" y2="279.4" width="0.1524" layer="91"/>
-<pinref part="X2" gate="G$1" pin="1"/>
+<pinref part="X3" gate="G$1" pin="1"/>
 <wire x1="76.2" y1="279.4" x2="71.12" y2="279.4" width="0.1524" layer="91"/>
 <wire x1="76.2" y1="276.86" x2="76.2" y2="279.4" width="0.1524" layer="91"/>

Commit message: Prototype ready for final review and manufacture
Parts:
- removed DT10: CGRM4001-G, diode:CGRM4001-G
- removed DT6, DT7: 16V, SparkFun-DiscreteSemi:DIODE-ZENER16V
- removed LED7: 3.3V, SparkFun-LED:LED-GREEN0603
- added D6: MBR0530, imix_v1:DIODESOD123
- added F5, F6: FIDUCIAL, GeekAmmo:FIDUCIAL
- added LED5: USER, SparkFun-LED:LED-BLUE0603
- added R30: 10K, SparkFun-Resistors:RESISTOR0603
- BAT1: device SparkFun-Electromechanical:BATTERY18650 -> imix_v1:BATTERY18650
- C10, C45, C8, C9, R11, R12, R4, R5, R6, R7, R8: value (none) -> DNP
- C11: value (none) -> 22pF
- C44, C46, C47, C7: value (none) -> 0.47uF
- C48: value (none) -> 4.7uF
- D1, D4: MPN (none) -> 610-1N759A
- D5: value DIODE-ZENER16V -> MBR0530; DKPN (none) -> MBR0530CT-ND
- L3: DKPN (none) -> 587-2045-1-ND; MFPN (none) -> LBR2012T100K
- LED3: value NRF -> 3.3V; device SparkFun-LED:LED-BLUE0603 -> SparkFun-LED:LED-GREEN0603
- LED4: value USER -> NRF
- R10, R13, R9: value (none) -> 10K
- R14: value (none) -> 2.2M
- R15: value (none) -> 160K
- U12: value TPS61040 -> 296-12686-1-ND; DKPN (none) -> 296-12686-1-ND
- U3: value AD712R -> TLV3202; DKPN (none) -> 296-34773-1-ND
- U4: value AD712R -> LM358
- renumbered DT5 to D4, DT9 to D5, U$2 to F1, U$3 to F3, U$5 to F4, U$6 to F2, U$7 to U12
Connections:
- net GND: now also LED5.C, R30.1; no longer LED7.C
- net N$29: now also LED5.A; no longer LED4.A
- net N$38: now also LED3.A; no longer LED7.A
- net N$43: now also D6.A; no longer DT10.A
- net N$51: no longer DT6.C
- net N$52: no longer DT7.C
- net N$75: now also LED4.A; no longer LED3.A
- net NOISE1: no longer DT6.A
- net NOISE2: no longer DT7.A
- net TRNG_EN: now also R30.2
- net VHIGH: now also D6.C; no longer DT10.C
Other:
- moved on the sheet: C11, C45, C46, C47, C49, R9
