File: hardware/v1_3/imix.brd (EAGLE design)
At the start: 87 x 102.5 mm, 154 parts, among them J2_3_5_AND_6 ARDUINO_R3NO_HOLES, SW1 TAC_SWITCHSMD, SW2 TAC_SWITCHSMD, U1 BQ2423X, U10 ISL29035, U11 FX0S8700CQ, U12 296-12686-1-ND, U13 SIP32401A, U14 SIP32401A, U15 SIP32401A, U16 SIP32401A, U17 74LVC4066BQ, U18 74LVC4066BQ, U3 TLV3202, U4 LM358, U5 LDO-TPS78233, U6 ATSAM4LCX_100, U8 SI7021, U9 NRF51422, X1 16MHz, X2 16MHz, X3 16MHz

Commit message: Down to 3 airwires
Routing:
- net VCC_SENSE_3V3: track 25.7 -> 82.6 mm
- net VCC_IN: track 85.5 -> 98.7 mm, vias 4 -> 5
- net VCC_MCU_3V3: track 68.3 -> 71.0 mm, vias 13 -> 14
Changed lines of the file:
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@@
 <layer number="18" name="Vias" color="2" fill="1" visible="yes" active="yes"/>
 <layer number="19" name="Unrouted" color="6" fill="1" visible="yes" active="yes"/>
-<layer number="20" name="Dimension" color="15" fill="1" visible="no" active="yes"/>
+<layer number="20" name="Dimension" color="15" fill="1" visible="yes" active="yes"/>
 <layer number="21" name="tPlace" color="7" fill="1" visible="yes" active="yes"/>
 <layer number="22" name="bPlace" color="7" fill="1" visible="yes" active="yes"/>
@@
 <layer number="28" name="bValues" color="7" fill="1" visible="no" active="yes"/>
 <layer number="29" name="tStop" color="7" fill="3" visible="yes" active="yes"/>
-<layer number="30" name="bStop" color="7" fill="6" visible="no" active="yes"/>
+<layer number="30" name="bStop" color="7" fill="6" visible="yes" active="yes"/>
 <layer number="31" name="tCream" color="7" fill="4" visible="no" active="yes"/>
 <layer number="32" name="bCream" color="7" fill="5" visible="no" active="yes"/>
@@
 <layer number="37" name="tTest" color="7" fill="1" visible="no" active="yes"/>
 <layer number="38" name="bTest" color="7" fill="1" visible="no" active="yes"/>
-<layer number="39" name="tKeepout" color="4" fill="11" visible="no" active="yes"/>
-<layer number="40" name="bKeepout" color="1" fill="11" visible="no" active="yes"/>
+<layer number="39" name="tKeepout" color="4" fill="11" visible="yes" active="yes"/>
+<layer number="40" name="bKeepout" color="1" fill="11" visible="yes" active="yes"/>
 <layer number="41" name="tRestrict" color="4" fill="10" visible="no" active="yes"/>
 <layer number="42" name="bRestrict" color="1" fill="10" visible="no" active="yes"/>
 <layer number="43" name="vRestrict" color="2" fill="10" visible="no" active="yes"/>
-<layer number="44" name="Drills" color="7" fill="1" visible="no" active="yes"/>
-<layer number="45" name="Holes" color="7" fill="1" visible="no" active="yes"/>
+<layer number="44" name="Drills" color="7" fill="1" visible="yes" active="yes"/>
+<layer number="45" name="Holes" color="7" fill="1" visible="yes" active="yes"/>
 <layer number="46" name="Milling" color="3" fill="1" visible="no" active="yes"/>
 <layer number="47" name="Measures" color="7" fill="1" visible="no" active="yes"/>
@@
 <layer number="50" name="dxf" color="7" fill="1" visible="no" active="no"/>
 <layer number="51" name="tDocu" color="14" fill="1" visible="no" active="yes"/>
-<layer number="52" name="bDocu" color="6" fill="1" visible="yes" active="yes"/>
+<layer number="52" name="bDocu" color="6" fill="1" visible="no" active="yes"/>
 <layer number="53" name="tGND_GNDA" color="7" fill="9" visible="no" active="no"/>
 <layer number="54" name="bGND_GNDA" color="1" fill="9" visible="no" active="no"/>
@@
 <layer number="152" name="_bDocu" color="7" fill="1" visible="no" active="yes"/>
 <layer number="153" name="FabDoc1" color="15" fill="1" visible="no" active="yes"/>
-<layer number="154" name="FabDoc2" color="15" fill="1" visible="yes" active="yes"/>
+<layer number="154" name="FabDoc2" color="15" fill="1" visible="no" active="yes"/>
 <layer number="155" name="FabDoc3" color="7" fill="1" visible="no" active="yes"/>
 <layer number="199" name="Contour" color="7" fill="1" visible="no" active="yes"/>
@@
 <wire x1="53.7" y1="63.1" x2="53.7" y2="58.6" width="0.1524" layer="15"/>
 <wire x1="56.45" y1="64.95" x2="56" y2="65.4" width="0.1524" layer="16"/>
-<wire x1="47.101040625" y1="27.89895625" x2="43.89895625" y2="23.89895625" width="0" layer="19" extent="1-1"/>
-<wire x1="27.5" y1="5.15" x2="22.86" y2="20.32" width="0" layer="19" extent="1-15"/>
-<wire x1="44.885" y1="4.48" x2="27.5" y2="5.15" width="0" layer="19" extent="1-1"/>
+<wire x1="43.89895625" y1="23.89895625" x2="42.6" y2="22.6" width="0.1524" layer="1"/>
+<wire x1="42.6" y1="22.6" x2="41.7" y2="22.6" width="0.1524" layer="1"/>
+<via x="41.7" y="22.6" extent="1-16" drill="0.3302"/>
+<wire x1="27.5" y1="5.15" x2="44.885" y2="4.48" width="0" layer="19" extent="1-1"/>
+<wire x1="22.86" y1="20.32" x2="27.5" y2="5.15" width="0" layer="19" extent="1-15"/>
 </signal>
 <signal name="USART3_RTS">
@@
 <wire x1="50.5" y1="29.70710625" x2="50.5" y2="28.5" width="0.1524" layer="1"/>
 <wire x1="50.5" y1="28.5" x2="48.5" y2="26.5" width="0.1524" layer="1"/>
-<wire x1="48.5" y1="26.5" x2="47.5" y2="26.5" width="0.1524" layer="1"/>
-<wire x1="47.5" y1="26.5" x2="46.101040625" y2="25.101040625" width="0.1524" layer="1"/>
-<wire x1="46.101040625" y1="25.101040625" x2="45.101040625" y2="25.101040625" width="0.1524" layer="1"/>
+<wire x1="48.5" y1="26.5" x2="46.5" y2="26.5" width="0.1524" layer="1"/>
+<wire x1="46.5" y1="26.5" x2="45.101040625" y2="25.101040625" width="0.1524" layer="1"/>
 </signal>
 <signal name="RF233_!RST">
@@
 <wire x1="74.5" y1="-4.6" x2="75.1" y2="-5.2" width="0.1524" layer="16"/>
 <wire x1="75.1" y1="-5.2" x2="76.1" y2="-5.2" width="0.1524" layer="16"/>
-<wire x1="74.75" y1="5.5" x2="22.88" y2="17.72" width="0" layer="19" extent="16-16"/>
+<wire x1="22.88" y1="17.72" x2="24.6" y2="16" width="0.4064" layer="15"/>
+<wire x1="24.6" y1="16" x2="33.8" y2="16" width="0.4064" layer="15"/>
+<wire x1="33.8" y1="16" x2="39.5" y2="10.3" width="0.4064" layer="15"/>
+<wire x1="39.5" y1="10.3" x2="45.2" y2="10.3" width="0.4064" layer="15"/>
+<wire x1="45.2" y1="10.3" x2="47.4" y2="8.1" width="0.4064" layer="15"/>
+<wire x1="47.4" y1="8.1" x2="68.9" y2="8.1" width="0.4064" layer="15"/>
+<wire x1="68.9" y1="8.1" x2="71.5" y2="5.5" width="0.4064" layer="15"/>
+<wire x1="71.5" y1="5.5" x2="74.75" y2="5.5" width="0.4064" layer="15"/>
 </signal>
 <signal name="GPIO2">
@@
 <wire x1="66.5" y1="52" x2="71.5" y2="47" width="0.1524" layer="1"/>
 <wire x1="33.5" y1="20.5" x2="32.1" y2="19.1" width="0.1524" layer="1"/>
-<wire x1="32.1" y1="19.1" x2="27.45" y2="14.45" width="0.1524" layer="1"/>
+<wire x1="32.1" y1="19.1" x2="27.05" y2="13.95" width="0.1524" layer="1"/>
 <contactref element="R5" pad="2"/>
 <wire x1="32.1" y1="20.55" x2="32.1" y2="19.1" width="0.1524" layer="1"/>
@@
 <contactref element="U18" pad="13"/>
 <contactref element="U18" pad="5"/>
-<wire x1="27.45" y1="14.45" x2="25.65" y2="14.45" width="0.1524" layer="1"/>
-<wire x1="25.65" y1="14.45" x2="25.6" y2="14.4" width="0.1524" layer="1"/>
-<via x="25.6" y="14.4" extent="1-16" drill="0.3302"/>
-<wire x1="25.6" y1="14.4" x2="24.8" y2="14.4" width="0.1524" layer="16"/>
-<wire x1="24.8" y1="14.4" x2="23.5" y2="13.1" width="0.1524" layer="16"/>
+<wire x1="27.05" y1="13.95" x2="25.25" y2="13.95" width="0.1524" layer="1"/>
+<wire x1="25.25" y1="13.95" x2="25.2" y2="13.9" width="0.1524" layer="1"/>
+<via x="25.2" y="13.9" extent="1-16" drill="0.3302"/>
+<wire x1="25.2" y1="13.9" x2="24.4" y2="13.9" width="0.1524" layer="16"/>
+<wire x1="24.4" y1="13.9" x2="23.5" y2="13.1" width="0.1524" layer="16"/>
 <wire x1="16.825" y1="15.1" x2="16.875" y2="15.15" width="0.1524" layer="16"/>
 <wire x1="68" y1="43.5" x2="71.5" y2="47" width="0.1524" layer="16"/>
@@
 <wire x1="9.505" y1="23.495" x2="9.505" y2="23.06" width="0.4064" layer="1"/>
 <contactref element="U1" pad="6"/>
-<wire x1="3.025" y1="53.25" x2="1.75" y2="53.25" width="0.1524" layer="1"/>
-<wire x1="1.75" y1="53.25" x2="1.5" y2="53.5" width="0.1524" layer="1"/>
-<wire x1="5.975" y1="52.25" x2="3.025" y2="53.25" width="0" layer="19" extent="1-1"/>
+<wire x1="3.025" y1="53.25" x2="2.975" y2="53.3" width="0.1524" layer="1"/>
+<wire x1="2.975" y1="53.3" x2="1.2" y2="53.3" width="0.1524" layer="1"/>
+<via x="1.2" y="53.3" extent="1-16" drill="0.3302"/>
+<wire x1="1.2" y1="53.3" x2="0.7" y2="52.8" width="0.1524" layer="16"/>
+<wire x1="0.7" y1="52.8" x2="0.7" y2="51.9" width="0.1524" layer="16"/>
+<wire x1="0.7" y1="51.9" x2="1.1" y2="51.5" width="0.1524" layer="16"/>
+<wire x1="1.1" y1="51.5" x2="10.1" y2="51.5" width="0.1524" layer="16"/>
+<wire x1="10.1" y1="51.5" x2="11.1" y2="50.5" width="0.1524" layer="16"/>
+<wire x1="11.1" y1="50.5" x2="11.5" y2="50.5" width="0.1524" layer="16"/>
 </signal>
 <signal name="N$47">
