File: hardware/v1_3/imix.brd (EAGLE design)
At the start: 87 x 102.5 mm, 156 parts, among them J2_3_5_AND_6 ARDUINO_R3NO_HOLES, SW1 TAC_SWITCHSMD, SW2 TAC_SWITCHSMD, U1 BQ2423X, U10 ISL29035, U11 FX0S8700CQ, U12 296-12686-1-ND, U13 SIP32401A, U14 SIP32401A, U15 SIP32401A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

Commit message: Attempts to fix mirrored footprints
Routing:
- net VHIGHSAMPLE: track 92.6 -> 81.6 mm
- net GND: track 225.4 -> 222.2 mm
Changed lines of the file:
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@@
 <wire x1="62" y1="-7.5" x2="63.07" y2="-8.57" width="0.1524" layer="1"/>
 <wire x1="63.07" y1="-8.57" x2="63.34" y2="-8.81" width="0.1524" layer="1"/>
-<wire x1="59.5" y1="28.75735625" x2="59.5" y2="29" width="0.1524" layer="1"/>
 <via x="83.5" y="27.3" extent="1-16" drill="0.3302"/>
 <via x="77" y="26.05" extent="1-16" drill="0.3302"/>
@@
 <via x="76.9" y="64" extent="1-16" drill="0.6"/>
 <wire x1="60.53553125" y1="28.42893125" x2="59.9644625" y2="29" width="0.1524" layer="1"/>
-<wire x1="59.9644625" y1="29" x2="59.5" y2="29" width="0.1524" layer="1"/>
-<wire x1="60.181978125" y1="28.075378125" x2="59.5" y2="28.75735625" width="0.1524" layer="1"/>
-<wire x1="59.5" y1="29" x2="59.5" y2="29.5" width="0.1524" layer="1"/>
 <wire x1="36.39895625" y1="29.39895625" x2="35.3" y2="28.3" width="0.4064" layer="1"/>
 <wire x1="49.27" y1="76.02" x2="48.02" y2="76.02" width="0.1524" layer="1"/>
@@
 <wire x1="57.35" y1="72.75" x2="57.8" y2="73.2" width="0.1524" layer="16"/>
 <via x="57.8" y="73.2" extent="1-16" drill="0.3302"/>
-<wire x1="48.825" y1="72.1" x2="47.4" y2="72.1" width="0.1524" layer="16"/>
 <via x="47.4" y="72.1" extent="1-16" drill="0.3302"/>
 <wire x1="46.735" y1="70.64" x2="46.735" y2="71.435" width="0.1524" layer="16"/>
@@
 <via x="53.2" y="30.55" extent="1-16" drill="0.3302"/>
 <wire x1="60.181978125" y1="28.075378125" x2="59.6" y2="28.65735625" width="0.1524" layer="1"/>
-<wire x1="59.6" y1="28.65735625" x2="59.6" y2="29.45" width="0.1524" layer="1"/>
+<wire x1="59.6" y1="28.65735625" x2="59.6" y2="28.95" width="0.1524" layer="1"/>
 <via x="59.6" y="29.45" extent="1-16" drill="0.3302"/>
+<wire x1="59.6" y1="28.95" x2="59.6" y2="29.45" width="0.1524" layer="1"/>
 <wire x1="83" y1="80.25" x2="84.95" y2="78.3" width="0.4064" layer="1"/>
 <wire x1="84.95" y1="78.3" x2="84.95" y2="77" width="0.4064" layer="1"/>
@@
 <wire x1="83.5" y1="75.55" x2="83.1" y2="75.55" width="0.4064" layer="1"/>
 <contactref element="LED1" pad="C"/>
+<wire x1="59.9644625" y1="29" x2="59.65" y2="29" width="0.1524" layer="1"/>
+<wire x1="59.65" y1="29" x2="59.6" y2="28.95" width="0.1524" layer="1"/>
 </signal>
 <signal name="SWDIO/TMS">
@@
 <wire x1="75" y1="33.5" x2="75" y2="35" width="0.1524" layer="1"/>
 <wire x1="62.2" y1="33.5" x2="75" y2="33.5" width="0.1524" layer="16"/>
-<wire x1="59.5" y1="27.5" x2="58.75" y2="28.25" width="0.1524" layer="1"/>
-<wire x1="59.5" y1="27.5" x2="59.474871875" y2="27.368271875" width="0.1524" layer="1"/>
 <via x="62.5" y="59.5" extent="1-16" drill="0.3302"/>
 <via x="76" y="42" extent="1-16" drill="0.3302"/>
@@
 <via x="62.2" y="33.5" extent="1-16" drill="0.3302"/>
 <wire x1="62.5" y1="56" x2="62.5" y2="59.5" width="0.1524" layer="1"/>
-<wire x1="58.75" y1="28.25" x2="58.75" y2="30" width="0.1524" layer="1"/>
+<wire x1="58.75" y1="28.09314375" x2="58.75" y2="30" width="0.1524" layer="1"/>
 <wire x1="58.75" y1="30" x2="62.25" y2="33.5" width="0.1524" layer="1"/>
 <wire x1="62.25" y1="33.5" x2="62.2" y2="33.5" width="0.1524" layer="1"/>
@@
 <wire x1="55.6" y1="62.2" x2="56.7" y2="61.1" width="0.1524" layer="16"/>
 <wire x1="56.7" y1="61.1" x2="60.9" y2="61.1" width="0.1524" layer="16"/>
+<wire x1="58.75" y1="28.09314375" x2="59.474871875" y2="27.368271875" width="0.1524" layer="1"/>
 </signal>
 <signal name="NRF_INT">
@@
 <wire x1="60.75" y1="25.75" x2="62.75" y2="25.75" width="0.1524" layer="16"/>
 <wire x1="62.75" y1="25.75" x2="64.425" y2="24.075" width="0.1524" layer="16"/>
-<wire x1="64.425" y1="24.075" x2="72.25" y2="16.25" width="0.1524" layer="16"/>
 <wire x1="60.45" y1="30.65" x2="64.1" y2="27" width="0.1524" layer="16"/>
 <wire x1="86.45" y1="75.05" x2="86.45" y2="56.05" width="0.1524" layer="1"/>
