File: hardware/v1_3/imix.sch (EAGLE design)
At the start: 151 parts, among them J2_3_5_AND_6 ARDUINO_R3NO_HOLES, Q2 AO3415, Q3 AO3415, Q4 AO3415, Q5 AO3415, U1 BQ2423X, U10 ISL29035, U11 FX0S8700CQ, U12 296-12686-1-ND, U3 TLV3202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

Commit message: Add 1K resistor b/n FTDI DTR and RESET. Closes #15
Parts:
- added R8: 1K, imix:RESISTOR0603-RES
Connections:
- new net DTR: J1.15, R8.2, U7.!DTR
- net !RESET: now also R8.1; no longer J1.15, U7.!DTR
Changed lines of the file:
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@@
 <part name="FRAME15" library="frames" deviceset="FRAME_A_L" device=""/>
 <part name="FRAME16" library="imix" deviceset="DOCFIELD" device="" value="True Random Number Generator (Lampert Circuit)"/>
+<part name="R8" library="imix" deviceset="RESISTOR" device="0603-RES" value="1K"/>
 </parts>
 <sheets>
@@
 <label x="210.82" y="86.36" size="1.778" layer="95"/>
 </segment>
-<segment>
-<wire x1="45.72" y1="121.92" x2="68.58" y2="121.92" width="0.1524" layer="91"/>
-<label x="48.26" y="121.92" size="1.778" layer="95"/>
-<pinref part="J1" gate="G$1" pin="15"/>
-</segment>
 </net>
 <net name="USART0_RX" class="0">
@@
 <wire x1="83.82" y1="116.84" x2="104.14" y2="116.84" width="0.1524" layer="91"/>
 <label x="96.52" y="116.84" size="1.778" layer="95"/>
+</segment>
+</net>
+<net name="DTR" class="0">
+<segment>
+<wire x1="45.72" y1="121.92" x2="68.58" y2="121.92" width="0.1524" layer="91"/>
+<label x="48.26" y="121.92" size="1.778" layer="95"/>
+<pinref part="J1" gate="G$1" pin="15"/>
 </segment>
 </net>
@@
 <instance part="FRAME6" gate="G$1" x="0" y="0"/>
 <instance part="FRAME12" gate="G$1" x="170.18" y="0"/>
+<instance part="R8" gate="G$1" x="147.32" y="121.92" rot="MR0"/>
 </instances>
 <busses>
@@
 </segment>
 </net>
+<net name="DTR" class="0">
+<segment>
+<pinref part="U7" gate="G$1" pin="!DTR"/>
+<wire x1="132.08" y1="121.92" x2="142.24" y2="121.92" width="0.1524" layer="91"/>
+<pinref part="R8" gate="G$1" pin="2"/>
+<label x="134.62" y="121.92" size="1.778" layer="95"/>
+</segment>
+</net>
 <net name="!RESET" class="0">
 <segment>
-<pinref part="U7" gate="G$1" pin="!DTR"/>
-<wire x1="132.08" y1="121.92" x2="154.94" y2="121.92" width="0.1524" layer="91"/>
-<label x="137.16" y="121.92" size="1.778" layer="95"/>
-</segment>
-</net>
+<pinref part="R8" gate="G$1" pin="1"/>
+<wire x1="152.4" y1="121.92" x2="165.1" y2="121.92" width="0.1524" layer="91"/>
+<label x="154.94" y="121.92" size="1.778" layer="95"/>
+</segment>
+</net>

Commit message: Fix power bugs and other issues in schematic
* Set EN1 on the battery charger to VCC
* Replaced the PMOS load switches with SIP32041As
* Added isolation for the I2C and the RF233 SPI busses
* Connected the I2C pullups to VCC_MCU, not VCC_SENSE
* Added resistor between FTDI DTR and RESET (previous commit)
* Moved power sense headers logically inward towards their power domains
Parts:
- removed Q2, Q3, Q4, Q5: AO3415, SparkFun-DiscreteSemi:MOSFET-PCHANNELDMG2307L
- added U13, U14, U15, U16: SIP32401A, shaneleonard-master-lbr:SIP32401A
- added U17, U18: 74LVC4066BQ, shaneleonard-master-lbr:74LVC4066BQ
Connections:
- removed net !NRF_PWR_EN: J3.7, Q5.G, R5.2, U6.PC17
- removed net !RF233_PWR_EN: J3.6, Q2.G, R6.2, U6.PC18
- removed net !SENSE_PWR_EN: J3.8, Q4.G, R4.2, U6.PC16
- removed net !TRNG_PWR_EN: Q3.G, R7.2, U6.PC19
- removed net N$14: J4.2.1, Q3.S, SJ7.2
- removed net N$36: J4.5.1, Q5.S, SJ2.2
- removed net N$37: J4.1.1, Q2.S, SJ3.2
- new net N$32: J4.2.1, SJ7.1, U16.OUT
- new net N$33: J4.1.1, SJ3.1, U15.OUT
- new net N$8: J4.4.1, SJ1.2, U13.OUT
- new net NRF_PWR_EN: J3.7, R5.2, U14.EN, U18.1E, U18.2E, U6.PC17
- new net NRF_TWI_SCL: U18.2Z, U9.P00
- new net NRF_TWI_SDA: U18.1Z, U9.P30
- new net RF233_CS: U17.4Z, U2.NSEL
- new net RF233_MISO: U17.1Z, U2.MISO
- new net RF233_MOSI: U17.2Z, U2.MOSI
- new net RF233_PWR_EN: J3.6, R6.2, U15.EN, U17.1E, U17.2E, U17.3E, U17.4E, U6.PC18
- new net RF233_SCK: U17.3Z, U2.SCLK
- new net SENSE_PWR_EN: J3.8, R4.2, U13.EN, U18.3E, U18.4E, U6.PC16
- new net SENSE_TWI_SCL: U10.SCL, U11.SCL/SCK, U18.4Z, U8.SCL
- new net SENSE_TWI_SDA: U10.SDA, U11.SDA/MOSI, U18.3Z, U8.SDA
- new net TRNG_PWR_EN: R7.2, U16.EN, U6.PC19
- net GND: now also R4.1, R5.1, R7.1, U13.GND, U14.GND, U15.GND, U16.GND, U17.GND, U18.GND
- net MISO: now also U17.1Y; no longer U2.MISO
- net MOSI: now also U17.2Y; no longer U2.MOSI
- net N$18: now also J4.5.1, SJ2.1, U14.OUT; no longer J4.4.1, Q4.S, SJ1.2
- net SCK: now also U17.3Y; no longer U2.SCLK
- net SPI_NCS3: now also U17.4Y; no longer U2.NSEL
- net TWI2_SCL: now also U18.2Y, U18.4Y; no longer U10.SCL, U11.SCL/SCK, U8.SCL, U9.P00
- net TWI2_SDA: now also U18.1Y, U18.3Y; no longer U10.SDA, U11.SDA/MOSI, U8.SDA, U9.P30
- net VCC_3V3: now also U13.IN, U14.IN, U15.IN, U16.IN; no longer J4.1.2, J4.2.2, J4.4.2, J4.5.2, R4.1, R5.1, R7.1, SJ1.1, SJ2.1, SJ3.1, SJ7.1
- net VCC_MCU_3V3: now also R25.2, R38.2, U17.VCC, U18.VCC
- net VCC_NRF_3V3: no longer Q5.D
- net VCC_RF233_3V3: now also J4.1.2, J4.5.2, SJ2.2, SJ3.2; no longer Q2.D
- net VCC_SENSE_3V3: now also J4.4.2, SJ1.1; no longer Q4.D, R25.2, R38.2
- net VCC_TRNG_3V3: now also J4.2.2, SJ7.2; no longer Q3.D
Other:
- moved on the sheet: D2, D3, D9, J4.1, J4.2, J4.3, J4.4, J4.5, R4, R5, R6, R7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

Commit message: Create PDF
Connections:
- net GND: no longer U1.EN1
- net VCC_IN: now also U1.EN1
Changed lines of the file:
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@@
 <junction x="48.26" y="58.42"/>
 <junction x="40.64" y="58.42"/>
-<wire x1="55.88" y1="78.74" x2="53.34" y2="78.74" width="0.1524" layer="91"/>
-<wire x1="53.34" y1="78.74" x2="53.34" y2="76.2" width="0.1524" layer="91"/>
 <junction x="53.34" y="63.5"/>
 <wire x1="53.34" y1="76.2" x2="53.34" y2="63.5" width="0.1524" layer="91"/>
 <wire x1="55.88" y1="76.2" x2="53.34" y2="76.2" width="0.1524" layer="91"/>
-<junction x="53.34" y="76.2"/>
 <pinref part="U1" gate="G$1" pin="!CE"/>
-<pinref part="U1" gate="G$1" pin="EN1"/>
 <pinref part="U1" gate="G$1" pin="EN2"/>
 <pinref part="U1" gate="G$1" pin="TMR"/>
@@
 <segment>
 <pinref part="C14" gate="G$1" pin="1"/>
-<wire x1="55.88" y1="86.36" x2="40.64" y2="86.36" width="0.1524" layer="91"/>
+<wire x1="55.88" y1="86.36" x2="53.34" y2="86.36" width="0.1524" layer="91"/>
+<wire x1="53.34" y1="86.36" x2="40.64" y2="86.36" width="0.1524" layer="91"/>
 <wire x1="40.64" y1="86.36" x2="38.1" y2="86.36" width="0.1524" layer="91"/>
 <junction x="40.64" y="86.36"/>
 <label x="38.1" y="86.36" size="1.778" layer="95" rot="R180" xref="yes"/>
 <pinref part="U1" gate="G$1" pin="IN"/>
-</segment>
-</net>
+<pinref part="U1" gate="G$1" pin="EN1"/>
+<wire x1="55.88" y1="78.74" x2="53.34" y2="78.74" width="0.1524" layer="91"/>
+<wire x1="53.34" y1="78.74" x2="53.34" y2="86.36" width="0.1524" layer="91"/>
+<junction x="53.34" y="86.36"/>
+</segment>
+</net>

Commit message: Eliminated FabDoc layers and migrated all components to imix library
Parts:
- removed RESET, USER: (no value), SparkFun-Retired:TAC_SWITCHSMD
- added SW1, SW2: TAC_SWITCHSMD, imix:TAC_SWITCHSMD
- B1: device stanford_iot_research:2450BM15A0015 -> imix:2450BM15A0015
- B2: device stanford_iot_research:BAL_NRF01D3 -> imix:BAL_NRF01D3
- BAT1: device imix_v1:BATTERY18650 -> imix:BATTERY18650
- C17: device rcl:C-EUC0603 -> imix:C-EUC0603
- D1, D4: device SparkFun-DiscreteSemi:DIODE-ZENERPTH -> imix:DIODE-ZENERPTH
- D2, D3, D9: value NSR1020MW2T3G -> 250mA/100V; device SparkFun-DiscreteSemi:BAT20JFILM -> imix:DIODEBAS16
- D5: device SparkFun-DiscreteSemi:DIODE-ZENER16V -> imix:DIODESOD123
- D6: device imix_v1:DIODESOD123 -> imix:DIODESOD123
- F1, F10, F2, F3, F4, F5, F6, F7, F8, F9: device GeekAmmo:FIDUCIAL -> imix:FIDUCIAL
- J1: device SparkFun-Connectors:M10X2ROUND_NOSILK -> imix:M10X2ROUND_NOSILK
- J2: device SparkFun-Connectors:M10NO_SILK_PTH_FEMALE -> imix:M10NO_SILK_PTH_FEMALE
- J3, J5: device SparkFun-Connectors:M08NO_SILK_FEMALE_PTH -> imix:M08NO_SILK_FEMALE_PTH
- J4.1, J4.2, J4.3, J4.4, J4.5: device SparkFun-Connectors:M02PTH -> imix:M021X02_NO_SILK
- J6: device SparkFun-Connectors:M06NO_SILK_FEMALE_PTH -> imix:M06NO_SILK_FEMALE_PTH
- L1: device stanford_iot_research:L -> imix:L
- L2: device stanford_iot_research:L1212 -> imix:L1212
- L3: device SparkFun-Passives:INDUCTOR0805 -> imix:INDUCTOR0805
- LED2: value 5V -> BLUE; device SparkFun-LED:LED-BLUE0603 -> imix:LED-BLUE0603
- LED3: value 3.3V -> BLUE; device SparkFun-LED:LED-GREEN0603 -> imix:LED-BLUE0603
- LED4: value NRF -> BLUE; device SparkFun-LED:LED-BLUE0603 -> imix:LED-BLUE0603
- LED5: value USER -> BLUE; device SparkFun-LED:LED-BLUE0603 -> imix:LED-BLUE0603
- TC1, TC2: device TagConnect:TC2030-IDC -> imix:TC2030-IDC
- U12: device SparkFun-PowerIC:TPS61040 -> imix:TPS61040
- U2: device stanford_iot_research:AT86RF233 -> imix:AT86RF233
- U3, U4: device analog-devices:AD712R -> imix:AD712R
- U5: device SparkFun-PowerIC:LDO-TPS78233 -> imix:LDO-TPS78233
- U7: device stanford_iot_research:FT231X -> imix:FT231X
- USB1, USB2: device SparkFun-Connectors-Fixed:USB-AB -> imix:USB-AB
- X1, X2, X3: device stanford_iot_research:XTAL_GROUNDED5X3.2MM -> imix:XTAL_GROUNDED5X3.2MM
Connections:
- net !RESET: now also SW1.3, SW1.4; no longer RESET.3, RESET.4
- net GND: now also SW1.1, SW1.2, SW2.1, SW2.2; no longer RESET.1, RESET.2, USER.1, USER.2
- net USER_BTN: now also SW2.3, SW2.4; no longer USER.3, USER.4
- net VCC_NRF_3V3: now also J4.5.2, SJ2.2
- net VCC_RF233_3V3: no longer J4.5.2, SJ2.2

Commit message: Passes DRC
Parts:
- C47, C48: device imix:C-EUC0603 -> imix:C-EUC0603-NOSILK
Changed lines of the file:
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@@
 <part name="GND38" library="SparkFun-Aesthetics" deviceset="GND" device=""/>
 <part name="C11" library="imix" deviceset="C-EU" device="C0603" value="22pF"/>
-<part name="C47" library="imix" deviceset="C-EU" device="C0603" value="0.47uF"/>
+<part name="C47" library="imix" deviceset="C-EU" device="C0603-NOSILK" value="0.47uF"/>
 <part name="GND33" library="SparkFun-Aesthetics" deviceset="GND" device=""/>
-<part name="C48" library="imix" deviceset="C-EU" device="C0603" value="4.7uF"/>
+<part name="C48" library="imix" deviceset="C-EU" device="C0603-NOSILK" value="4.7uF"/>
 <part name="GND40" library="SparkFun-Aesthetics" deviceset="GND" device=""/>
 <part name="C49" library="imix" deviceset="CAP_POL" device="C" value="10uF"/>

Commit message: Rearranged analog pins according to #16
Connections:
- net ADCIFE0: now also U6.PA04; no longer U6.PA05
- net ADCIFE1: now also U6.PA05; no longer U6.PA07
- net ADCIFE2: now also U6.PA07; no longer U6.PB02
- net ADCIFE3: now also U6.PB02; no longer U6.PB03
- net ADCIFE4: now also U6.PB03; no longer U6.PB04
- net ADCIFE5: now also U6.PB04; no longer U6.PB05
- net GPIO8: now also U6.PA20; no longer U6.PC25
- net LIGHT_!INT: now also U6.PC25; no longer U6.PA04
- net VHIGHSAMPLE: now also U6.PB05

Commit message: Fab/assembly documentation for v1.3
Parts:
- added LED1: (no value), imix:LED-BLUE0603
- added R19: 1K, imix:RESISTOR0603-RES
- LED2, LED3, LED4, LED5: value BLUE -> (none)
Connections:
- new net KERNEL_LED: R19.1, U6.PC22
- new net N$14: LED1.A, R19.2
- net GND: now also LED1.C
Changed lines of the file:
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@@
 <attributes>
 <attribute name="AUTHOR" value="Shane Leonard"/>
-<attribute name="REVISION" value="1.2"/>
+<attribute name="REVISION" value="1.3"/>
 </attributes>
 <variantdefs>
@@
 <part name="R2" library="imix" deviceset="RESISTOR" device="0603-RES" value="4.7K"/>
 <part name="R24" library="imix" deviceset="RESISTOR" device="0603-RES" value="1K"/>
-<part name="LED5" library="imix" deviceset="LED-BLUE" device="0603" value="BLUE"/>
+<part name="LED5" library="imix" deviceset="LED-BLUE" device="0603"/>
 <part name="GND18" library="SparkFun-Aesthetics" deviceset="DGND" device=""/>
 <part name="SW2" library="imix" deviceset="TAC_SWITCH" device="SMD" value="TAC_SWITCHSMD"/>
@@
 <part name="GND22" library="SparkFun-Aesthetics" deviceset="DGND" device=""/>
 <part name="R21" library="imix" deviceset="RESISTOR" device="0603-RES" value="1K"/>
-<part name="LED3" library="imix" deviceset="LED-BLUE" device="0603" value="BLUE"/>
+<part name="LED3" library="imix" deviceset="LED-BLUE" device="0603"/>
 <part name="GND39" library="SparkFun-Aesthetics" deviceset="DGND" device=""/>
 <part name="D9" library="imix" deviceset="DIODE" device="BAS16" value="250mA/100V"/>
@@
 <part name="U6" library="imix" deviceset="ATSAM4LCX_100" device=""/>
 <part name="R20" library="imix" deviceset="RESISTOR" device="0603-RES" value="1K"/>
-<part name="LED2" library="imix" deviceset="LED-BLUE" device="0603" value="BLUE"/>
+<part name="LED2" library="imix" deviceset="LED-BLUE" device="0603"/>
 <part name="C14" library="imix" deviceset="C-EU" device="C0603" value="1uF"/>
 <part name="R18" library="imix" deviceset="RESISTOR" device="0603-RES" value="DNP"/>
@@
 <part name="GND49" library="SparkFun-Aesthetics" deviceset="GND" device=""/>
 <part name="R34" library="imix" deviceset="RESISTOR" device="0603-RES" value="1K"/>
-<part name="LED4" library="imix" deviceset="LED-BLUE" device="0603" value="BLUE"/>
+<part name="LED4" library="imix" deviceset="LED-BLUE" device="0603"/>
 <part name="GND35" library="SparkFun-Aesthetics" deviceset="DGND" device=""/>
 <part name="J2_3_5_AND_6" library="imix" deviceset="ARDUINO_R3" device="NO_HOLES"/>
@@
 <part name="U18" library="shaneleonard-master-lbr" deviceset="74LVC4066" device="BQ"/>
 <part name="GND66" library="SparkFun-Aesthetics" deviceset="DGND" device=""/>
+<part name="R19" library="imix" deviceset="RESISTOR" device="0603-RES" value="1K"/>
+<part name="LED1" library="imix" deviceset="LED-BLUE" device="0603"/>
+<part name="GND67" library="SparkFun-Aesthetics" deviceset="DGND" device=""/>
 </parts>
 <sheets>
@@
 <attribute name="VALUE" x="165.481" y="143.764" size="1.778" layer="96" rot="R180"/>
 </instance>
-<instance part="SW1" gate="S" x="213.36" y="157.48" rot="MR90"/>
+<instance part="SW1" gate="S" x="213.36" y="157.48" smashed="yes" rot="MR90">
+<attribute name="NAME" x="219.71" y="154.94" size="1.778" layer="95" rot="MR90"/>
+</instance>
 <instance part="R33" gate="G$1" x="210.82" y="175.26" rot="R90"/>
 <instance part="GND7" gate="G$1" x="15.24" y="78.74"/>
@@
 <instance part="LED5" gate="G$1" x="152.4" y="38.1"/>
 <instance part="GND18" gate="G$1" x="152.4" y="30.48"/>
-<instance part="SW2" gate="S" x="248.92" y="157.48" rot="MR90"/>
+<instance part="SW2" gate="S" x="248.92" y="157.48" smashed="yes" rot="MR90">
+<attribute name="NAME" x="255.27" y="154.94" size="1.778" layer="95" rot="MR90"/>
+</instance>
 <instance part="GND37" gate="G$1" x="246.38" y="144.78"/>
 <instance part="R3" gate="G$1" x="246.38" y="175.26" rot="R90"/>
@@
 <instance part="FRAME1" gate="G$1" x="0" y="0"/>
 <instance part="FRAME2" gate="G$1" x="170.18" y="0"/>
+<instance part="R19" gate="G$1" x="50.8" y="55.88" rot="MR270"/>
+<instance part="LED1" gate="G$1" x="50.8" y="45.72"/>
+<instance part="GND67" gate="G$1" x="50.8" y="35.56"/>
 </instances>
 <busses>
@@
 <wire x1="81.28" y1="88.9" x2="83.82" y2="88.9" width="0.1524" layer="91"/>
 </segment>
+<segment>
+<pinref part="GND67" gate="G$1" pin="GND"/>
+<pinref part="LED1" gate="G$1" pin="C"/>
+<wire x1="50.8" y1="38.1" x2="50.8" y2="40.64" width="0.1524" layer="91"/>
+</segment>
 </net>
 <net name="SWDIO/TMS" class="0">
@@
 </segment>
 </net>
+<net name="N$14" class="0">
+<segment>
+<pinref part="LED1" gate="G$1" pin="A"/>
+<pinref part="R19" gate="G$1" pin="2"/>
+<wire x1="50.8" y1="48.26" x2="50.8" y2="50.8" width="0.1524" layer="91"/>
+</segment>
+</net>
+<net name="KERNEL_LED" class="0">
+<segment>
+<pinref part="R19" gate="G$1" pin="1"/>
+<pinref part="U6" gate="G$1" pin="PC22"/>
+<wire x1="50.8" y1="60.96" x2="83.82" y2="60.96" width="0.1524" layer="91"/>
+<label x="60.96" y="60.96" size="1.778" layer="95"/>
+</segment>
+</net>
