File: hardware/v1_2/imix.brd (EAGLE design)
At the start: 87 x 102.5 mm, 151 parts, among them J2_3_5_AND_6 ARDUINO_R3NO_HOLES, Q2 AO3415, Q3 AO3415, Q4 AO3415, Q5 AO3415, U1 BQ2423X, U10 ISL29035, U11 FX0S8700CQ, U12 296-12686-1-ND, U3 TLV3202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

Commit message: Correct ADC numbering in doc. Closes #16
Connections:
- removed net ADCIFE0: J2_3_5_AND_6.A0, U6.25
- new net ADCIFE6: J2_3_5_AND_6.A5, U6.29
- net ADCIFE1: now also J2_3_5_AND_6.A0, U6.25; no longer J2_3_5_AND_6.A1, U6.31
- net ADCIFE2: now also J2_3_5_AND_6.A1, U6.31; no longer J2_3_5_AND_6.A2, U6.22
- net ADCIFE3: now also J2_3_5_AND_6.A2, U6.22; no longer J2_3_5_AND_6.A3, U6.23
- net ADCIFE4: now also J2_3_5_AND_6.A3, U6.23; no longer J2_3_5_AND_6.A4, U6.28
- net ADCIFE5: now also J2_3_5_AND_6.A4, U6.28; no longer J2_3_5_AND_6.A5, U6.29
Routing:
- net ADCIFE6: track 0.00 -> 30.3 mm, vias 0 -> 1
- net ADCIFE0: track 21.1 -> 0.00 mm, vias 1 -> 0
- net ADCIFE2: track 31.2 -> 22.7 mm
- net ADCIFE4: track 28.4 -> 34.8 mm
- net ADCIFE3: track 34.8 -> 31.2 mm
- net ADCIFE5: track 30.3 -> 28.4 mm
- net ADCIFE1: track 22.7 -> 21.1 mm
Changed lines of the file:
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@@
 <wire x1="31.6" y1="30.3" x2="36.4" y2="35.2" width="0.1524" layer="1"/>
 </signal>
-<signal name="ADCIFE0">
+<signal name="ADCIFE1">
 <contactref element="U6" pad="25"/>
 <contactref element="J2_3_5_AND_6" pad="A0"/>
@@
 <wire x1="56" y1="24.75" x2="56.25" y2="24.5" width="0.1524" layer="1"/>
 </signal>
-<signal name="ADCIFE1">
+<signal name="ADCIFE2">
 <contactref element="U6" pad="31"/>
 <contactref element="J2_3_5_AND_6" pad="A1"/>
@@
 <wire x1="62" y1="22.5" x2="61.5" y2="22" width="0.1524" layer="1"/>
 </signal>
-<signal name="ADCIFE2">
+<signal name="ADCIFE3">
 <contactref element="U6" pad="22"/>
 <contactref element="J2_3_5_AND_6" pad="A2"/>
@@
 <wire x1="54" y1="25.25" x2="54" y2="25.5" width="0.1524" layer="16"/>
 </signal>
-<signal name="ADCIFE3">
+<signal name="ADCIFE4">
 <contactref element="U6" pad="23"/>
 <contactref element="J2_3_5_AND_6" pad="A3"/>
@@
 <wire x1="54.75" y1="23" x2="54" y2="23.75" width="0.1524" layer="16"/>
 </signal>
-<signal name="ADCIFE4">
+<signal name="ADCIFE5">
 <contactref element="U6" pad="28"/>
 <contactref element="J2_3_5_AND_6" pad="A4"/>
@@
 <wire x1="60.428928125" y1="25" x2="61.25" y2="25" width="0.1524" layer="1"/>
 </signal>
-<signal name="ADCIFE5">
+<signal name="ADCIFE6">
 <contactref element="U6" pad="29"/>
 <contactref element="J2_3_5_AND_6" pad="A5"/>
